File: Schematic/Actuator_v2/Actuator_v2.kicad_sch (KiCad schematic)
At the start: 15 parts, among them J1 12V Power in, J2 12V Actuator out, Q1 BC547C, Q2 BUZ11, U1 Heltec_Wifi_LoRa_V1, U1 TSR_1-2450

Commit message: New layout by Eenesh
Parts:
- D1: footprint (none) -> LED_THT:LED_D5.0mm_IRGrey
- J1, J2: footprint (none) -> TerminalBlock_RND:TerminalBlock_RND_205-00001_1x02_P5.00mm_Horizontal
- JP1: footprint (none) -> Connector_PinHeader_2.54mm:PinHeader_1x02_P2.54mm_Vertical
- JP2: footprint (none) -> Connector_PinHeader_2.54mm:PinHeader_1x03_P2.54mm_Vertical
- R1, R2, R3, R4, R5, R6: footprint (none) -> Resistor_THT:R_Axial_DIN0411_L9.9mm_D3.6mm_P12.70mm_Horizontal
- U1: footprint (none) -> Heltec_Wifi_Lora_v1:Heltec_WiFi_LoRa_V1
- renumbered U1 to U2
Connections:
- no-connect marks 0 -> 27
